Commit message: urdf

File: src/vehicle_description/urdf/macro.xacro (robot description, xacro)
@@ -23,8 +23,8 @@
       <type>transmission_interface/SimpleTransmission</type>
       <joint name="${name}">
-        <hardwareInterface>hardware_interface/EffortJointInterface</hardwareInterface>
+        <hardwareInterface>VelocityJointInterface</hardwareInterface>
       </joint>
       <actuator name="motor_${name}">
-        <hardwareInterface>hardware_interface/EffortJointInterface</hardwareInterface>
+        <hardwareInterface>VelocityJointInterface</hardwareInterface>
         <mechanicalReduction>1</mechanicalReduction>
       </actuator>
@@ -51,114 +51,4 @@
       </actuator>
     </transmission>
-  </xacro:macro>
-  <!-- DELIRO CHASIS LINK MACRO -->
-  <xacro:macro name="base_link" params="name origin_xyz origin_rpy">
-    <link name="${name}">
-      <visual>
-        <origin rpy="${origin_rpy}" xyz="${origin_xyz}" />
-        <geometry>
-          <mesh filename="package://deliro_description/meshes/Chasis/DeliRo_Chasis.dae"/>
-        </geometry>
-      </visual>
-      <collision>
-        <origin rpy="${origin_rpy}" xyz="${origin_xyz}" />
-        <geometry>
-          <box size="0.684 1 0.416" />
-        </geometry>
-      </collision>
-      <inertial>
-        <mass value="10" />
-        <origin rpy="${origin_rpy}" xyz="${origin_xyz}" />
-        <inertia ixx="1.0" ixy="0" ixz="0" iyy="1.0" iyz="0" izz="1.0" />
-      </inertial>
-    </link>
-  </xacro:macro>
-  <!-- DELIRO HEAD LINK MACRO -->
-  <xacro:macro name="head" params="name origin_xyz origin_rpy">
-    <link name="${name}">
-      <visual>
-        <origin rpy="${origin_rpy}" xyz="${origin_xyz}" />
-        <geometry>
-          <mesh filename="package://deliro_description/meshes/Head/DeliRo_Head.dae"/>
-        </geometry>
-      </visual>
-      <collision>
-        <origin rpy="${origin_rpy}" xyz="${origin_xyz}" />
-        <geometry>
-          <box size="0.711 0.348 0.621" />
-        </geometry>
-      </collision>
-      <inertial>
-        <mass value="15" />
-        <origin rpy="${origin_rpy}" xyz="${origin_xyz}" />
-        <inertia ixx="1.0" ixy="0" ixz="0" iyy="1.0" iyz="0" izz="1.0" />
-      </inertial>
-    </link>
-  </xacro:macro>
-  <!-- DELIRO TRUCK LINK MACRO -->
-  <xacro:macro name="truck" params="name origin_xyz origin_rpy">
-    <link name="${name}">
-      <visual>
-        <origin rpy="${origin_rpy}" xyz="${origin_xyz}" />
-        <geometry>
-          <mesh filename="package://deliro_description/meshes/Truck/DeliRo_Truck.dae"/>
-        </geometry>
-      </visual>
-      <collision>
-        <origin rpy="${origin_rpy}" xyz="${origin_xyz}" />
-        <geometry>
-          <mesh filename="package://deliro_description/meshes/Truck/DeliRo_Truck.dae"/>
-        </geometry>
-      </collision>
-      <inertial>
-        <mass value="10" />
-        <origin rpy="${origin_rpy}" xyz="${origin_xyz}" />
-        <inertia ixx="1.0" ixy="0" ixz="0" iyy="1.0" iyz="0" izz="1.0" />
-      </inertial>
-    </link>
-  </xacro:macro>
-  <!-- DELIRO LOCKER LINK MACRO -->
-  <xacro:macro name="locker" params="name origin_xyz origin_rpy">
-    <link name="${name}">
-      <visual>
-        <origin rpy="${origin_rpy}" xyz="${origin_xyz}" />
-        <geometry>
-          <mesh filename="package://deliro_description/meshes/Locker/DeliRo_Locker.dae"/>
-        </geometry>
-      </visual>
-      <collision>
-        <origin rpy="${origin_rpy}" xyz="${origin_xyz}" />
-        <geometry>
-          <box size="0.662 0.616 0.57" />
-        </geometry>
-      </collision>
-      <inertial>
-        <mass value="12" />
-        <origin rpy="${origin_rpy}" xyz="${origin_xyz}" />
-        <inertia ixx="1.0" ixy="0" ixz="0" iyy="1.0" iyz="0" izz="1.0" />
-      </inertial>
-    </link>
-  </xacro:macro>
-  <!-- DELIRO WHEEL LINK MACRO -->
-  <xacro:macro name="wheel" params="name origin_xyz origin_rpy">
-    <link name="${name}">
-      <visual>
-        <origin rpy="${origin_rpy}" xyz="${origin_xyz}" />
-        <geometry>
-          <mesh filename="package://deliro_description/meshes/Wheel/wheel.dae"/>
-        </geometry>
-      </visual>
-      <collision>
-        <origin rpy="${origin_rpy}" xyz="${origin_xyz}" />
-        <geometry>
-          <mesh filename="package://deliro_description/meshes/Wheel/wheel.dae"/>
-        </geometry>
-      </collision>
-      <inertial>
-        <mass value="3" />
-        <origin rpy="0.7854 0 0" xyz="${origin_xyz}" />
-        <inertia ixx="1.0" ixy="0" ixz="0" iyy="1.0" iyz="0" izz="1.0" />
-      </inertial>
-    </link>
   </xacro:macro>
   <!-- //////////////////////////////////////////// USEFUL MACROS //////////////////////////////////////////// -->

File: src/vehicle_description/urdf/robot_parameters.xacro (robot description, xacro)
@@ -1,11 +1,11 @@
 <?xml version="1.0" ?>
 <robot xmlns:xacro="http://www.ros.org/wiki/xacro">
-  <xacro:property name="Robot_Base" value="deliro_base" />
+  <xacro:property name="Robot_Base" value="vehicle_base" />
   <xacro:property name="FR_wheel" value="front_right_wheel" />
   <xacro:property name="FL_wheel" value="front_left_wheel" />
   <xacro:property name="BR_wheel" value="backward_right_wheel" />
   <xacro:property name="BL_wheel" value="backward_left_wheel" />
-  <xacro:property name="Robot_head" value="deliro_head" />
-  <xacro:property name="Locker_box" value="deliro_locker" />
-  <xacro:property name="Truck" value="deliro_truck" />
+  <xacro:property name="Robot_head" value="vehicle_head" />
+  <xacro:property name="Locker_box" value="vehicle_locker" />
+  <xacro:property name="Truck" value="vehicle_truck" />
 </robot>

File: src/vehicle_description/urdf/simple_vehicle.xacro (robot description, xacro)
@@ -1,8 +1,7 @@
 <?xml version="1.0" ?>
-<robot name="DeliRo" xmlns:xacro="http://ros.org/wiki/xacro">
-    <xacro:arg name="use_truck" default="false"/>
-    <xacro:include filename="$(find deliro_description)/urdf/macro.xacro" />
-    <xacro:include filename="$(find deliro_description)/urdf/robot_parameters.xacro" />
-    <xacro:include filename="$(find deliro_description)/urdf/deliro.gazebo" />
+<robot name="SVehicle" xmlns:xacro="http://ros.org/wiki/xacro">
+    <xacro:include filename="$(find vehicle_description)/urdf/macro.xacro" />
+    <xacro:include filename="$(find vehicle_description)/urdf/robot_parameters.xacro" />
+    <xacro:include filename="$(find vehicle_description)/urdf/simple_vehicle.gazebo" />
     <!-- //////////////////// GENERAL STRUCTURE //////////////////// -->
     <!-- BASEFOOTPRINT (Dummy baselink) -->
@@ -12,27 +11,11 @@
         origin_rpy="0 0 0" origin_xyz="0 0 0"
         parent="base_footprint" child="${Robot_Base}"/>
-    <!-- CHASIS -->
-    <xacro:base_link name = "${Robot_Base}" origin_rpy="0 0 0" origin_xyz="0 0 0"/>
-    <!-- HEAD -->
-    <xacro:fix_joint name="${Robot_Base}__${Robot_head}"
-        axis_xyz="0 0 1"
-        origin_rpy="0 0 0" origin_xyz="0 -0.3100 0.1850"
-        parent="${Robot_Base}" child="${Robot_head}"/>
-    <xacro:head name = "${Robot_head}" origin_rpy="0 0 0" origin_xyz="0 0 0.2637"/>
-    <!-- CHOOSE BETWEEN LOCKERS OR TRUCK (Default = Locker) -->
-    <xacro:if value="$(arg use_truck)">
-        <xacro:fix_joint name="${Robot_Base}__${Truck}"
-            axis_xyz="0 0 1"
-            origin_rpy="0 0 0" origin_xyz="0 0.1733 0.1850"
-            parent="${Robot_Base}" child="${Truck}"/>
-        <xacro:truck name ="${Truck}" origin_rpy="0 0 0" origin_xyz="0 0 0.1970"/>
-    </xacro:if>
-    <xacro:unless value="$(arg use_truck)">
-        <xacro:fix_joint name="${Robot_Base}__${Locker_box}"
-            axis_xyz="0 0 1"
-            origin_rpy="0 0 0" origin_xyz="0 0.1733 0.1850"
-            parent="${Robot_Base}" child="${Locker_box}"/>
-        <xacro:locker name ="${Locker_box}" origin_rpy="0 0 0" origin_xyz="0 0 0.2800"/>
-    </xacro:unless>
+    <xacro:m_link_box name="${Robot_Base}"
+        origin_rpy="0 0 0" origin_xyz="0 0 0"
+        size="0.616 0.662 0.57"
+        mass="15"
+        ixx="1.0" ixy="0" ixz="0"
+        iyy="1.0" iyz="0"
+        izz="1.0"/>
     <!-- ////////////////// GENERAL STRUCTURE END //////////////////// -->
     <!-- //////////////////// WHEELS STRUCTURE 0.30241 //////////////////// -->
@@ -43,5 +26,4 @@
         parent="${Robot_Base}" child="${FL_wheel}_Bearing"
         limit_e="1000" limit_l="-0.785" limit_u="0.785" limit_v="0.5" />
-    <!--<link name="${FL_wheel}_Bearing"/>-->
     <xacro:m_link_box name="${FL_wheel}_Bearing"
         origin_rpy="0 0 0" origin_xyz="0 0 0"
@@ -56,5 +38,11 @@
         parent="${FL_wheel}_Bearing" child="${FL_wheel}"
         limit_e="1000" limit_v="0.5"/>
-    <xacro:wheel name = "${FL_wheel}" origin_rpy="0 0 0" origin_xyz="0 0 0"/>
+    <xacro:m_link_cylinder name="${FL_wheel}"
+        origin_rpy="1.5708 0 0" origin_xyz="0 0 0"
+        radius="0.12" length="0.103"
+        mass="5"
+        ixx="1.0" ixy="0" ixz="0"
+        iyy="1.0" iyz="0"
+        izz="1.0" />
     <!-- FRONT RIGHT WHEEL-->
     <xacro:rev_joint name="${FR_wheel}__Steer"
@@ -63,5 +51,4 @@
         parent="${Robot_Base}" child="${FR_wheel}_Bearing"
         limit_e="1000" limit_l="-0.785" limit_u="0.785" limit_v="0.5" />
-    <!--<link name="${FR_wheel}_Bearing"/>-->
     <xacro:m_link_box name="${FR_wheel}_Bearing"
         origin_rpy="0 0 0" origin_xyz="0 0 0"
@@ -76,5 +63,11 @@
         parent="${FR_wheel}_Bearing" child="${FR_wheel}"
         limit_e="1000" limit_v="0.5"/>
-    <xacro:wheel name = "${FR_wheel}" origin_rpy="0 0 3.14159" origin_xyz="0 0 0"/>
+    <xacro:m_link_cylinder name="${FR_wheel}"
+        origin_rpy="1.5708 0 0" origin_xyz="0 0 0"
+        radius="0.12" length="0.103"
+        mass="5"
+        ixx="1.0" ixy="0" ixz="0"
+        iyy="1.0" iyz="0"
+        izz="1.0" />
     <!-- BACK LEFT WHEEL-->
     <xacro:cont_joint name="${BL_wheel}__Rear"
@@ -83,5 +76,11 @@
         parent="${Robot_Base}" child="${BL_wheel}"
         limit_e="1000" limit_v="0.5"/>
-    <xacro:wheel name = "${BL_wheel}" origin_rpy="0 0 0" origin_xyz="0 0 0"/>
+    <xacro:m_link_cylinder name="${BL_wheel}"
+        origin_rpy="1.5708 0 0" origin_xyz="0 0 0"
+        radius="0.12" length="0.103"
+        mass="5"
+        ixx="1.0" ixy="0" ixz="0"
+        iyy="1.0" iyz="0"
+        izz="1.0" />
     <!-- BACK RIGHT WHEEL-->
     <xacro:cont_joint name="${BR_wheel}__Rear"
@@ -90,5 +89,11 @@
         parent="${Robot_Base}" child="${BR_wheel}"
         limit_e="1000" limit_v="0.5"/>
-    <xacro:wheel name = "${BR_wheel}" origin_rpy="0 0 3.14159" origin_xyz="0 0 0"/>
+    <xacro:m_link_cylinder name="${BR_wheel}"
+        origin_rpy="1.5708 0 0" origin_xyz="0 0 0"
+        radius="0.12" length="0.103"
+        mass="5"
+        ixx="1.0" ixy="0" ixz="0"
+        iyy="1.0" iyz="0"
+        izz="1.0" />
     <!-- //////////////////// WHEELS STRUCTURE END //////////////////// -->
 </robot>
